File: PCB/EAGLE/projects/TBCP V0.1/Schematic.sch (EAGLE design)
At the start: 76 parts, among them J1 12 Supply, J2 TB Header, J3 FP Header, U1 ESP32-DEVKITC, U2 TLE9201SG, U3 LM7805_TO220V

Commit message: Fix's to TBCP V0.1 hardware
Parts:
- removed E57: DPADS_PAD-0400-S, 52101-101-REV-A_v16:DPADS_PAD-0400-S
- removed SJ1: (no value), jumper:SJ2W
- removed SJ3, SJ4: (no value), jumper:SJ2WW
Connections:
- removed net HBRIDGE_MISO: SJ3.2, U2.SO
- removed net HBRIDGE_MOSI: SJ1.2, U2.SI
- removed net HBRIDGE_SPI_CLOCK: SJ4.2, U2.SCK
- net 0VDC: now also U2.!CS, U2.SCK, U2.SI, U2.SO; no longer SJ1.1, SJ3.1, SJ4.1
- net M0-: no longer E57.P
- net SPI_CLOCK: no longer SJ4.3
- net SPI_CS: no longer U2.!CS
- net SPI_MISO: no longer SJ3.3
- net SPI_MOSI: no longer SJ1.3
Other:
- note removed: "Solder jumps To select SPI Mode"
- moved on the sheet: C1, C2, E1, E10, E11, E12, E13, E14, E15, E16, E17, E18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
