File: PCB/EAGLE/projects/TBCP V0.1/Schematic.brd (EAGLE design)
At the start: 160.6 x 99.4 mm, 76 parts, among them J1 12 Supply, J2 TB Header, J3 FP Header, U1 ESP32-DEVKITC, U2 TLE9201SG, U3 LM7805_TO220V

Commit message: Fix's to TBCP V0.1 hardware
Parts:
- removed E57: DPADS_PAD-0400-S, 52101-101-REV-A_v16:DPADS_0400-S
- removed SJ1: (no value), jumper:SJ_2
- removed SJ3, SJ4: (no value), jumper:SJ_2W
- moved J1 43.2 mm to (148.6, 54.6), turned to 90 degrees
- moved E56 17.0 mm to (83.2, 36.8)
- moved U2 14.5 mm to (97.8, 38.1), turned to 0 degrees
- moved C1 12.8 mm to (83.8, 3.81)
- moved C2 12.8 mm to (58.4, 3.81)
- moved U3 12.8 mm to (71.1, 1.27)
Connections:
- removed net HBRIDGE_MISO: SJ3.2, U2.3
- removed net HBRIDGE_MOSI: SJ1.2, U2.8
- removed net HBRIDGE_SPI_CLOCK: SJ4.2, U2.10
- net 0VDC: now also U2.10, U2.3, U2.8, U2.9; no longer SJ1.1, SJ3.1, SJ4.1
- net M0-: no longer E57.PAD
- net SPI_CLOCK: no longer SJ4.3
- net SPI_CS: no longer U2.9
- net SPI_MISO: no longer SJ3.3
- net SPI_MOSI: no longer SJ1.3
Routing:
- net SPI_CS: track 82.2 -> 3.81 mm
- net SPI_MOSI: track 69.0 -> 3.81 mm
- net HBRDIGE_DISABLE: track 3.81 -> 68.0 mm
- net SPI_CLOCK: track 48.5 -> 3.81 mm
- net HBRIDGE_SPI_CLOCK: track 34.4 -> 0.00 mm
- net 12VDC: track 127.1 -> 161.1 mm
- net HBRIDGE_MOSI: track 33.4 -> 0.00 mm
- net SPI_MISO: track 32.5 -> 3.81 mm
- net 0VDC: track 26.5 -> 54.4 mm
- net HBRIDGE_DIRECTION: track 51.2 -> 29.4 mm
- net VPFB2: track 29.1 -> 48.7 mm
- net HBRIDGE_MISO: track 19.5 -> 0.00 mm
- net N$1: track 30.5 -> 13.2 mm
- net PPFB-SCALED: track 24.8 -> 38.7 mm
- net M0-: track 22.8 -> 36.0 mm
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Other:
- board text added: "Project: Throttle Body Control Platform By: Oliver Bell, Piyapat Srisawat Date: 21/07/2024 Verison: 0.1"
- board text removed: "---------"
- board text removed: "---------------"
- board text removed: "Project: Throttle Body Control Platform By: Oliver Bell, Piyapat Srisawat Date: 14/06/2024 Verison: 0.1"
