File: PCB/EAGLE/projects/TBCP V2/Schematic.brd (EAGLE design)
At the start: 160 x 71.1 mm, 110 parts, among them J1 12 Supply, J2 TB Header, J3 FP Header, Q1 DMP4025LK3Q-13, U1 ESP32-DEVKITC, U100 ADS1115, U101 TLE9201SG, U2 7805

Commit message: Added 3d Models to headers
Parts:
- S1, S2, S3, S4: value MOMENTARY-SWITCH-SPST-PTH-6.0MM-KIT -> MOMENTARY-SWITCH-SPST; device SparkFun-Switches:TACTILE_SWITCH_PTH_6.0MM_KIT -> 12mm TAC SWITCH:TACTILE_SWITCH_PTH_6.0MM
Changed lines of the file:
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@@
 </layers>
 <board>
+<fusionsync huburn="a.YnVzaW5lc3M6Z21haWw1NDMxMjA" projecturn="a.YnVzaW5lc3M6Z21haWw1NDMxMjAjMjAyNDA4MDI3ODc4NDU4NTY" f3durn="urn:adsk.wipprod:dm.lineage:snQFJ72zQ7GlnnzWu_bt0Q" pcbguid="" lastpulledtime="" lastsyncedchangeguid="" latestrevisionid="24751035-2efd-4e9c-881c-419d906286fd" lastsyncedrevisionid="24751035-2efd-4e9c-881c-419d906286fd" lastboardhashguid="3e8b2e3c-fb25-53c3-6edb-7b2b26c3eb37" lastpushedtime="2024-08-04T09:28:40Z" linktopcb3d="true"/>
 <plain>
 <text x="30.48" y="24.13" size="0.8128" layer="25" ratio="15" rot="R270" align="center-left">EN</text>
@@
 </element>
 <element name="U$1" library="Wintec Logo" package="WINTEC" value="WINTEC" x="111.76" y="29.21" smashed="yes"/>
-<element name="S5" library="500SSP1S1M6QEA" package="500SSP1S1M6QEA" value="500SSP1S1M6QEA" x="83.82" y="5.08" smashed="yes" rot="R90">
-<attribute name="DESCRIPTION" value="SLIDE, 5A, 120VAC/28VDC SPDT, On-On Through Hole, Right Angle" x="83.82" y="5.08" size="1.778" layer="27" rot="R90" display="off"/>
-<attribute name="ELEMENT14_PART_NUMBER" value="" x="83.82" y="5.08" size="1.778" layer="27" rot="R90" display="off"/>
-<attribute name="ELEMENT14_PRICE-STOCK" value="" x="83.82" y="5.08" size="1.778" layer="27" rot="R90" display="off"/>
-<attribute name="HEIGHT" value="6mm" x="83.82" y="5.08" size="1.778" layer="27" rot="R90" display="off"/>
-<attribute name="MANUFACTURER_NAME" value="E-Switch" x="83.82" y="5.08" size="1.778" layer="27" rot="R90" display="off"/>
-<attribute name="MANUFACTURER_PART_NUMBER" value="500SSP1S1M6QEA" x="83.82" y="5.08" size="1.778" layer="27" rot="R90" display="off"/>
+<element name="S5" library="500SSP1S1M6QEA" package="500SSP1S1M6QEA" package3d_urn="urn:adsk.eagle:package:45039936/2" value="500SSP1S1M6QEA" x="83.82" y="5.08" smashed="yes" rot="R90">
 <attribute name="NAME" x="73.66" y="11.43" size="1.016" layer="25" ratio="15" rot="R180" align="bottom-center"/>
 <attribute name="VALUE" x="83.82" y="5.08" size="1.27" layer="27" ratio="15" rot="R90" align="center"/>
 </element>
-<element name="S4" library="SparkFun-Switches" library_urn="urn:adsk.eagle:library:535" package="TACTILE_SWITCH_PTH_6.0MM_KIT" package3d_urn="urn:adsk.eagle:package:40170/2" value="MOMENTARY-SWITCH-SPST-PTH-6.0MM-KIT" x="49.53" y="7.62" smashed="yes">
+<element name="S4" library="12mm TAC SWITCH" package="TACTILE_SWITCH_PTH_6.0MM" package3d_urn="urn:adsk.eagle:package:45039953/2" value="MOMENTARY-SWITCH-SPST" x="49.53" y="7.62" smashed="yes">
 <attribute name="NAME" x="49.53" y="3.175" size="1.016" layer="25" font="vector" ratio="15" align="bottom-center"/>
-<attribute name="PROD_ID" value="SWCH-08441" x="49.53" y="7.62" size="1.778" layer="27" display="off"/>
-<attribute name="SF_SKU" value="COM-00097 " x="49.53" y="7.62" size="1.778" layer="27" display="off"/>
 <attribute name="VALUE" x="49.53" y="4.445" size="0.6096" layer="27" font="vector" ratio="20" align="top-center"/>
 </element>
-<element name="S1" library="SparkFun-Switches" library_urn="urn:adsk.eagle:library:535" package="TACTILE_SWITCH_PTH_6.0MM_KIT" package3d_urn="urn:adsk.eagle:package:40170/2" value="MOMENTARY-SWITCH-SPST-PTH-6.0MM-KIT" x="19.05" y="7.62" smashed="yes">
+<element name="S1" library="12mm TAC SWITCH" package="TACTILE_SWITCH_PTH_6.0MM" package3d_urn="urn:adsk.eagle:package:45039953/2" value="MOMENTARY-SWITCH-SPST" x="19.05" y="7.62" smashed="yes">
 <attribute name="NAME" x="19.05" y="3.175" size="1.016" layer="25" font="vector" ratio="15" align="bottom-center"/>
-<attribute name="PROD_ID" value="SWCH-08441" x="19.05" y="7.62" size="1.778" layer="27" display="off"/>
-<attribute name="SF_SKU" value="COM-00097 " x="19.05" y="7.62" size="1.778" layer="27" display="off"/>
 <attribute name="VALUE" x="19.05" y="4.445" size="0.6096" layer="27" font="vector" ratio="20" align="top-center"/>
 </element>
-<element name="S2" library="SparkFun-Switches" library_urn="urn:adsk.eagle:library:535" package="TACTILE_SWITCH_PTH_6.0MM_KIT" package3d_urn="urn:adsk.eagle:package:40170/2" value="MOMENTARY-SWITCH-SPST-PTH-6.0MM-KIT" x="29.21" y="7.62" smashed="yes">
+<element name="S2" library="12mm TAC SWITCH" package="TACTILE_SWITCH_PTH_6.0MM" package3d_urn="urn:adsk.eagle:package:45039953/2" value="MOMENTARY-SWITCH-SPST" x="29.21" y="7.62" smashed="yes">
 <attribute name="NAME" x="29.21" y="3.175" size="1.016" layer="25" font="vector" ratio="15" align="bottom-center"/>
-<attribute name="PROD_ID" value="SWCH-08441" x="24.13" y="7.62" size="1.778" layer="27" display="off"/>
-<attribute name="SF_SKU" value="COM-00097 " x="24.13" y="7.62" size="1.778" layer="27" display="off"/>
 <attribute name="VALUE" x="29.21" y="4.445" size="0.6096" layer="27" font="vector" ratio="20" align="top-center"/>
 </element>
-<element name="S3" library="SparkFun-Switches" library_urn="urn:adsk.eagle:library:535" package="TACTILE_SWITCH_PTH_6.0MM_KIT" package3d_urn="urn:adsk.eagle:package:40170/2" value="MOMENTARY-SWITCH-SPST-PTH-6.0MM-KIT" x="39.37" y="7.62" smashed="yes">
+<element name="S3" library="12mm TAC SWITCH" package="TACTILE_SWITCH_PTH_6.0MM" package3d_urn="urn:adsk.eagle:package:45039953/2" value="MOMENTARY-SWITCH-SPST" x="39.37" y="7.62" smashed="yes">
 <attribute name="NAME" x="39.37" y="3.175" size="1.016" layer="25" font="vector" ratio="15" align="bottom-center"/>
-<attribute name="PROD_ID" value="SWCH-08441" x="34.29" y="7.62" size="1.778" layer="27" display="off"/>
-<attribute name="SF_SKU" value="COM-00097 " x="34.29" y="7.62" size="1.778" layer="27" display="off"/>
 <attribute name="VALUE" x="39.37" y="4.445" size="0.6096" layer="27" font="vector" ratio="20" align="top-center"/>
 </element>
@@
 <wire x1="67.31" y1="10.16" x2="66.04" y2="10.16" width="1" layer="16"/>
 <wire x1="67.31" y1="10.16" x2="68.58" y2="10.16" width="1" layer="16"/>
+<wire x1="130.81" y1="54.61" x2="138.43" y2="54.61" width="0" layer="19" extent="1-1"/>
+<wire x1="118.11" y1="54.19" x2="128.27" y2="54.61" width="0" layer="19" extent="1-1"/>
+<wire x1="107.95" y1="54.61" x2="118.11" y2="54.19" width="0" layer="19" extent="1-1"/>
+<wire x1="102.87" y1="52.92" x2="107.95" y2="52.92" width="0" layer="19" extent="1-1"/>
+<wire x1="93.98" y1="57.15" x2="102.87" y2="54.61" width="0" layer="19" extent="1-1"/>
+<wire x1="82.55" y1="59.69" x2="93.98" y2="60.96" width="0" layer="19" extent="16-16"/>
+<wire x1="80.01" y1="47.3075" x2="82.55" y2="59.69" width="0" layer="19" extent="16-16"/>
+<wire x1="81.28" y1="44.45" x2="80.01" y2="47.3075" width="0" layer="19" extent="16-16"/>
+<wire x1="77.47" y1="41.91" x2="78.105" y2="44.45" width="0" layer="19" extent="16-16"/>
+<wire x1="69.85" y1="40.64" x2="70.64375" y2="40.64" width="0" layer="19" extent="16-16"/>
+<wire x1="64.77" y1="46.99" x2="68.35" y2="45.615" width="0" layer="19" extent="16-16"/>
+<wire x1="67.35" y1="35.665" x2="64.77" y2="39.37" width="0" layer="19" extent="16-16"/>
+<wire x1="59.69" y1="46.99" x2="64.77" y2="46.99" width="0" layer="19" extent="1-1"/>
+<wire x1="60.97" y1="27.94" x2="58.42" y2="36.83" width="0" layer="19" extent="16-16"/>
+<wire x1="91.44" y1="38.1" x2="81.28" y2="44.45" width="0" layer="19" extent="16-16"/>
+<wire x1="97.79" y1="33.02" x2="91.44" y2="38.1" width="0" layer="19" extent="1-1"/>
+<wire x1="97.79" y1="24.13" x2="97.79" y2="31.38" width="0" layer="19" extent="1-1"/>
+<wire x1="94.715" y1="24.13" x2="97.79" y2="24.13" width="0" layer="19" extent="1-1"/>
+<wire x1="97.79" y1="16.88" x2="97.79" y2="24.13" width="0" layer="19" extent="1-1"/>
+<wire x1="81.28" y1="19.05" x2="94.715" y2="24.13" width="0" layer="19" extent="1-1"/>
+<wire x1="68.58" y1="11.43" x2="81.28" y2="19.05" width="0" layer="19" extent="1-1"/>
+<wire x1="49.53" y1="7.62" x2="66.04" y2="8.89" width="0" layer="19" extent="1-1"/>
+<wire x1="46.14" y1="12.7" x2="49.53" y2="7.62" width="0" layer="19" extent="1-1"/>
+<wire x1="39.37" y1="7.62" x2="44.45" y2="12.7" width="0" layer="19" extent="1-1"/>
+<wire x1="35.98" y1="12.7" x2="39.37" y2="7.62" width="0" layer="19" extent="1-1"/>
+<wire x1="29.21" y1="7.62" x2="34.29" y2="12.7" width="0" layer="19" extent="1-1"/>
+<wire x1="25.82" y1="12.7" x2="29.21" y2="7.62" width="0" layer="19" extent="1-1"/>
+<wire x1="19.05" y1="7.62" x2="24.13" y2="12.7" width="0" layer="19" extent="1-1"/>
+<wire x1="15.66" y1="12.7" x2="19.05" y2="7.62" width="0" layer="19" extent="1-1"/>
+<wire x1="43.19" y1="53.34" x2="59.69" y2="46.99" width="0" layer="19" extent="1-1"/>
+<wire x1="27.94" y1="55.88" x2="43.18" y2="55.88" width="0" layer="19" extent="1-1"/>
+<wire x1="115.57" y1="10.16" x2="97.79" y2="15.24" width="0" layer="19" extent="1-1"/>
+<wire x1="4.03" y1="33.02" x2="13.97" y2="12.7" width="0" layer="19" extent="1-1"/>
+<wire x1="4.03" y1="36.83" x2="4.03" y2="33.02" width="0" layer="19" extent="1-1"/>
+<wire x1="4.03" y1="40.64" x2="4.03" y2="36.83" width="0" layer="19" extent="1-1"/>
+<wire x1="4.03" y1="44.45" x2="4.03" y2="40.64" width="0" layer="19" extent="1-1"/>
+<wire x1="4.03" y1="48.26" x2="4.03" y2="44.45" width="0" layer="19" extent="1-1"/>
+<wire x1="4.03" y1="52.07" x2="4.03" y2="48.26" width="0" layer="19" extent="1-1"/>
+<wire x1="148.59" y1="12.7" x2="115.57" y2="10.16" width="0" layer="19" extent="1-1"/>
 </signal>
 <signal name="12VDC">
@@
 </note>
 <note version="8.3" severity="warning">
+Since Version 8.3, EAGLE supports Fusion synchronisation.
+This feature will not be available in this version and saving
+the document will break the link to the Fusion PCB feature.
+</note>
+<note version="8.3" severity="warning">

Commit message: Added First Case Prototype
Parts:
- moved C1 2.54 mm to (94.0, 35.6)
Routing:
- net 12VDC: track 147.4 -> 152.4 mm
Changed lines of the file:
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@@
 <layer number="45" name="Holes" color="7" fill="1" visible="no" active="yes"/>
 <layer number="46" name="Milling" color="3" fill="1" visible="no" active="yes"/>
-<layer number="47" name="Measures" color="7" fill="1" visible="yes" active="yes"/>
+<layer number="47" name="Measures" color="7" fill="1" visible="no" active="yes"/>
 <layer number="48" name="Document" color="7" fill="1" visible="no" active="yes"/>
 <layer number="49" name="Reference" color="7" fill="1" visible="no" active="yes"/>
@@
 </autorouter>
 <elements>
-<element name="C1" library="BeagleBone_Blue_R3" library_urn="urn:adsk.eagle:library:5828899" package="TAP5-80" package3d_urn="urn:adsk.eagle:package:5829687/1" override_package3d_urn="urn:adsk.eagle:package:45070000/2" override_package_urn="urn:adsk.eagle:footprint:5829245/1" value="" x="91.44" y="35.56" smashed="yes" rot="R90">
-<attribute name="NAME" x="86.106" y="32.512" size="1.27" layer="25" ratio="15" rot="R90"/>
-<attribute name="VALUE" x="94.488" y="33.274" size="1.27" layer="27" ratio="10" rot="R90"/>
+<element name="C1" library="BeagleBone_Blue_R3" library_urn="urn:adsk.eagle:library:5828899" package="TAP5-80" package3d_urn="urn:adsk.eagle:package:5829687/1" override_package3d_urn="urn:adsk.eagle:package:45070000/2" override_package_urn="urn:adsk.eagle:footprint:5829245/1" value="" x="93.98" y="35.56" smashed="yes" rot="R90">
+<attribute name="NAME" x="88.646" y="32.512" size="1.27" layer="25" ratio="15" rot="R90"/>
+<attribute name="VALUE" x="97.028" y="33.274" size="1.27" layer="27" ratio="10" rot="R90"/>
 </element>
 <element name="D6" library="Wurth_LEDs_WL-SMCW" library_urn="urn:adsk.eagle:library:19028156" package="WL-SMCW_0805" package3d_urn="urn:adsk.eagle:package:19028167/5" value="150080AS75000" x="5.08" y="33.02" smashed="yes">
@@
 <wire x1="69.35" y1="34.6075" x2="69.35" y2="35.665" width="0.65" layer="16"/>
 <polygon width="0.000009375" layer="16" isolate="0.254">
-<vertex x="91.44" y="31.90875"/>
+<vertex x="93.98" y="31.90875"/>
 <vertex x="71.4375" y="31.90875"/>
 <vertex x="69.05625" y="34.29"/>
@@
 <vertex x="80.3275" y="33.9725"/>
 <vertex x="81.12125" y="34.76625"/>
-<vertex x="90.805" y="34.76625"/>
-<vertex x="91.44" y="34.13125"/>
+<vertex x="93.50375" y="34.76625"/>
+<vertex x="93.98" y="34.29"/>
 </polygon>
 <wire x1="83.82" y1="19.05" x2="83.82" y2="18.68" width="1.5" layer="1"/>
@@
 <wire x1="107.561" y1="9.265" x2="110.865" y2="9.265" width="0.508" layer="1"/>
 <wire x1="83.82" y1="29.21" x2="87.63" y2="33.02" width="2.54" layer="1"/>
-<wire x1="87.63" y1="33.02" x2="91.44" y2="33.02" width="2.54" layer="1"/>
+<wire x1="87.63" y1="33.02" x2="93.98" y2="33.02" width="2.54" layer="1"/>
 <wire x1="83.82" y1="21.59" x2="83.82" y2="29.21" width="2.54" layer="1"/>
-<wire x1="91.44" y1="33.02" x2="90.805" y2="33.02" width="2.1" layer="16"/>
-<wire x1="91.44" y1="33.02" x2="91.44" y2="32.0675" width="0.3048" layer="16"/>
-<wire x1="91.44" y1="33.02" x2="91.44" y2="33.9725" width="0.3048" layer="16"/>
-<wire x1="90.17" y1="33.02" x2="91.44" y2="33.02" width="0.3048" layer="16"/>
+<wire x1="93.98" y1="33.02" x2="93.345" y2="33.02" width="2.1" layer="16"/>
+<wire x1="93.98" y1="33.02" x2="93.98" y2="32.0675" width="0.3048" layer="16"/>
+<wire x1="93.98" y1="33.02" x2="93.98" y2="33.9725" width="0.3048" layer="16"/>
+<wire x1="90.17" y1="33.02" x2="93.98" y2="33.02" width="0.3048" layer="16"/>
 <wire x1="86.36" y1="33.02" x2="86.36" y2="34.29" width="0.4064" layer="16"/>
 <wire x1="86.36" y1="34.29" x2="86.36" y2="34.925" width="0.4064" layer="16"/>
